Commit message: Cross-check pass: fix grasp geometry, odom topic, Nav2 wiring
Bugs found and fixed while reviewing the whole simulation:
- Gripper fingers extended in -z while the tool/grasp frame was at +z, so
  IK placed the tool at the can but the fingers pointed away. Fingers now
  extend +z (verified: IK reaches all tray/shelf targets at 0 cm residual
  with the tool pointing straight down).
- diff_drive_controller publishes /diff_drive_controller/odom, not /odom;
  fixed the mission subscription and Nav2 odom_topic.
- Base now does a precise rotate-then-drive alignment (bidirectional) so
  both Nav2 and odom backends end at the exact picking pose, keeping the
  fixed arm/collision geometry valid; tracks odom yaw for this.
- Nav2: replaced the navigation_launch.py include + topic relay with
  explicit servers so the controller cmd_vel is deterministically remapped
  onto the diff-drive controller; added the required bt_navigator
  'navigators' block.
- MoveIt: guard plan() result with a success check before executing, and
  wrap MoveItConfigsBuilder so a config error degrades to the direct
  backend instead of killing the launch.
- Docker: add Mesa software-GL (headless sensor rendering), drop unused
  topic_tools.

https://claude.ai/code/session_01CuHJ3oP9Vu4yKiUgoco3Xk

File: 03-place-items-on-shelf/01-simulation/shelf_ws/src/shelf_description/urdf/robot.urdf.xacro (robot description, xacro)
@@ -171,14 +171,16 @@
     <origin xyz="0 0 0.11"/>
   </joint>
-  <!-- parallel fingers (prismatic, along y, extending down in -z) -->
+  <!-- parallel fingers (prismatic, along y). They extend in +z — the same
+       distal direction as the tool frame — so when the wrist points the tool
+       down at a can, the fingers straddle it (tool tip sits between them). -->
   <xacro:macro name="finger" params="name sign">
     <link name="${name}">
       <visual>
-        <origin xyz="0 0 -0.05"/>
+        <origin xyz="0 0 0.05"/>
         <geometry><box size="0.02 0.02 0.10"/></geometry>
         <material name="metal"/>
       </visual>
       <collision>
-        <origin xyz="0 0 -0.05"/>
+        <origin xyz="0 0 0.05"/>
         <geometry><box size="0.02 0.02 0.10"/></geometry>
       </collision>
